Commit message: [Add] avp demo with mujoco (fixed orientation + weld)

File: fr3_husky_description/mjcf/dual_fr3_husky.xml.xacro (robot description, xacro)
@@ -96,4 +96,5 @@
             finger_vis_mesh_materials="['off_white','black']">
             <cam_body>
+                <body name="${arm_prefix}_fr3_hand_tcp" pos="0 0 0.1034"/>
                 <xacro:if value="$(arg with_realsense)">
                     <xacro:realsense_d435i_mjcf prefix="${arm_prefix}" ee2cam_tf="${ee2cam_tf}"
@@ -146,4 +147,10 @@
                  width="300" height="300" mark="edge" markrgb="0.8 0.8 0.8" />
         <material name="groundplane" texture="groundplane" texuniform="true" texrepeat="5 5" reflectance="0.2" />
+        <material name="table_brown" rgba="0.55 0.27 0.07 1" />
+        <material name="env_red" rgba="1 0.072272 0.039546 1" />
+        <material name="env_blue" rgba="0.024157 0.445201 0.737911 1" />
+        <material name="ring_gray" rgba="0.85 0.85 0.85 1" />
+        <mesh name="table_mesh" file="$(find fr3_husky_description)/meshes/table.stl" scale="0.5 0.5 0.4" />
+        <mesh name="bowl_mesh" file="$(find fr3_husky_description)/meshes/cup_nohandle.stl" scale="1.2 1.2 0.05" />
         <xacro:fr3_assets arm_id="$(arg arm_id)"/>
         <xacro:franka_hand_assets/>
@@ -161,4 +168,22 @@
         <!-- ground plane -->
         <geom name="floor" type="plane" size="0 0 0.05" material="groundplane" />
+        <!-- Environment objects from tmm_mujoco/robots/dual_fr3_husky_env.xml -->
+        <geom name="table" type="mesh" mesh="table_mesh" material="table_brown" pos="1 -0.3 0" />
+        <body name="blue_bowl_body" pos="0.8 -0.6 0.555">
+            <geom name="blue_bowl_geom" type="mesh" mesh="bowl_mesh" material="env_blue" mass="0.2" />
+        </body>
+        <body name="red_bowl_body" pos="0.8 0.0 0.555">
+            <geom name="red_bowl_geom" type="mesh" mesh="bowl_mesh" material="env_red" mass="0.2" />
+        </body>
+        <body name="blue_cylinder_body" pos="0.8 -0.3 0.56">
+            <freejoint name="blue_cylinder_free" />
+            <geom name="blue_cylinder_geom" type="cylinder" size="0.03 0.03" material="env_blue" mass="0.05" />
+            <!-- Square ring fixed to the cylinder top. Ring plane is X-Z, so the hole normal is global Y. -->
+            <!-- <geom name="blue_cylinder_ring_top" type="box" pos="0 0 0.105" size="0.04 0.005 0.005" material="ring_gray" mass="0.005" />
+            <geom name="blue_cylinder_ring_bottom" type="box" pos="0 0 0.035" size="0.04 0.005 0.005" material="ring_gray" mass="0.005" />
+            <geom name="blue_cylinder_ring_left" type="box" pos="-0.035 0 0.07" size="0.005 0.005 0.035" material="ring_gray" mass="0.005" />
+            <geom name="blue_cylinder_ring_right" type="box" pos="0.035 0 0.07" size="0.005 0.005 0.035" material="ring_gray" mass="0.005" /> -->
+            <!-- <geom name="blue_cylinder_handle" type="box" pos="0 0 0.05" size="0.02 0.002 0.02" material="env_blue" mass="0.005" /> -->
+        </body>
         <body name="root" pos="0 0 0">
             <joint name="world_joint" type="free" stiffness="0" damping="0" frictionloss="0" armature="0" />
@@ -192,4 +217,8 @@
         </body>
     </worldbody>
+    <equality>
+        <weld name="weld_blue_right_tcp" body1="right_fr3_hand_tcp" body2="blue_cylinder_body"
+              active="false" solref="0.02 1" solimp="0.9 0.95 0.001"/>
+    </equality>
     <!-- Wheel actuators -->
     <xacro:husky_wheel_actuator prefix="" as_two_wheels="false"/>
