Commit message: edit scene xml.  move table position and obj position

File: fr3_husky_description/mjcf/coffee_scene.xml.xacro (robot description, xacro)
@@ -6,5 +6,5 @@
               group="1" name="wall_rear_visual" material="walls_mat"/> -->
         <!-- TableArena-style table with coffee task dimensions -->
-        <body name="coffee_table" pos="0.74 -0.25 0.6">
+        <body name="coffee_table" pos="0.9 -0.05 0.6">
             <geom name="coffee_table_collision"
                   pos="0 0 0"
@@ -56,5 +56,5 @@
         </body>
         <!-- Coffee machine, matching the CoffeeMachineObject composition in mimicgen -->
-        <body name="coffee_machine_root" pos="0.74 -0.1 0.75" quat="0 0 0 1">
+        <body name="coffee_machine_root" pos="0.74 0.0 0.75" quat="0 0 0 1">
             <!-- <freejoint name="coffee_machine_joint"/> -->
             <body name="coffee_machine_body_root" pos="0 -0.05 0" quat="0 0 0 1">
@@ -204,5 +204,5 @@
         </body>
         <!-- Coffee pod, which is the manipulated object -->
-        <body name="obj" pos="0.68 -0.4 0.7" quat="1 0 0 0"> <!-- z-axis : 1 0 0 0 | y-axis : NONE | x-axis : 1 0 0 0 -->
+        <body name="obj" pos="0.68 -0.3 0.7" quat="1 0 0 0"> <!-- z-axis : 1 0 0 0 | y-axis : NONE | x-axis : 1 0 0 0 -->
             <freejoint name="obj_joint"/>
             <geom name="coffee_pod_g0"

File: fr3_husky_description/mjcf/dual_fr3_husky.xml.xacro (robot description, xacro)
@@ -153,4 +153,6 @@
         <mesh name="table_mesh" file="$(find fr3_husky_description)/meshes/table.stl" scale="0.5 0.5 0.4" />
         <mesh name="bowl_mesh" file="$(find fr3_husky_description)/meshes/cup_nohandle.stl" scale="1.2 1.2 0.05" />
+        <texture file="$(find fr3_husky_description)/textures/ceramic.png" type="cube" name="tex-ceramic"/>
+        <material name="table_ceramic" reflectance="0.0" shininess="0.0" specular="0.2" texrepeat="1 1" texture="tex-ceramic"/>
         <!-- matte object -->
         <texture file="$(find fr3_husky_description)/textures/cement.png" type="2d" name="tex-cement"/>
@@ -181,12 +183,12 @@
         <geom name="floor" type="plane" size="0 0 0.05" material="groundplane" />
         <!-- Environment objects from tmm_mujoco/robots/dual_fr3_husky_env.xml -->
-        <geom name="table" type="mesh" mesh="table_mesh" material="table_brown" pos="1 -0.3 0" />
-        <body name="blue_bowl_body" pos="0.68 -0.6 0.555">
+        <geom name="table" type="mesh" mesh="table_mesh" material="table_ceramic" pos="1 -0.05 0" />
+        <body name="blue_bowl_body" pos="0.75 -0.4 0.555">
             <geom name="blue_bowl_geom" type="mesh" mesh="bowl_mesh" material="obj_blue" mass="0.2" />
         </body>
-        <body name="red_bowl_body" pos="0.68 0.0 0.555">
+        <body name="red_bowl_body" pos="0.75 0.2 0.555">
             <geom name="red_bowl_geom" type="mesh" mesh="bowl_mesh" material="obj_red" mass="0.2" />
         </body>
-        <body name="obj" pos="0.68 -0.3 0.62">
+        <body name="obj" pos="0.78 0.14 0.62">
             <freejoint name="obj_joint"/>
             <!-- <geom name="blue_cylinder_geom" type="cylinder" size="0.03 0.03" material="env_blue" mass="0.05" /> -->

File: fr3_husky_description/mjcf/square_scene.xml.xacro (robot description, xacro)
@@ -7,8 +7,8 @@
               group="1" name="wall_rear_visual" material="walls_mat"/> -->
         <!-- Table geometry from robosuite TableArena with NutAssembly dimensions -->
-        <body name="table" pos="0.7 -0.25 0.6">
+        <body name="table" pos="0.9 -0.05 0.6">
             <geom name="table_collision"
                   pos="0 0 0"
-                  size="0.4 0.6 0.025"
+                  size="0.35 0.5 0.025"
                   type="box"
                   group="0"
@@ -16,5 +16,5 @@
             <geom name="table_visual"
                   pos="0 0 0"
-                  size="0.4 0.6 0.025"
+                  size="0.35 0.5 0.025"
                   type="box"
                   conaffinity="0"
@@ -57,5 +57,5 @@
         </body>
         <!-- Fixed square-task peg -->
-        <body name="peg1" pos="0.7 -0.15 0.65">
+        <body name="peg1" pos="0.8 -0.05 0.65">
             <geom pos="0 0 0"
                   size="0.020 0.020 0.15"
@@ -72,6 +72,6 @@
         </body>
         <!-- Square nut from robosuite square-nut.xml --> <!-- z-axis : 0.7071 0 0 -0.7071 | y-axis : 0.7071 0 0 -0.7071 | x-axis : 0.7071 0 0 -0.7071 -->
-        <body name="obj" pos="0.7 -0.5 0.84" quat="0.7071 0 0 -0.7071">
-            <joint name="obj_joint" type="free" damping="0.0005"/>
+        <body name="obj" pos="0.72 -0.3 0.62" quat="0.7071 0 0 -0.7071">
+            <freejoint name="obj_joint"/>
             <geom pos="-0.03325 0 0"
                   size="0.0105 0.04375 0.02"

File: fr3_husky_description/mjcf/threading_scene.xml.xacro (robot description, xacro)
@@ -14,8 +14,8 @@
                   conaffinity="0"/>
         </body>
-        <body name="threading_table" pos="0.8 -0.25 0.7">
+        <body name="threading_table" pos="0.8 -0.05 0.7">
             <geom name="threading_table_top"
                   type="box"
-                  size="0.26 0.6 0.02"
+                  size="0.26 0.5 0.02"
                   material="table_ceramic"
                   friction="1 0.005 0.0001"/>

File: fr3_husky_description/mjcf/threepieceassembly_scene.xml.xacro (robot description, xacro)
@@ -23,5 +23,5 @@
              - piece_2: 4-layer bridge piece, unit half-size 0.02
              Placement here is deterministic and chosen to sit on the FR3 Husky top plate. -->
-        <body name="threepieceassembly_table" pos="0.9 -0.25 0.6">
+        <body name="threepieceassembly_table" pos="0.9 -0.05 0.6">
             <geom name="threepieceassembly_table_top"
                   type="box"
@@ -33,5 +33,5 @@
                   solimp="0.9 0.95 0.001"/>
         </body>
-        <body name="base" pos="0.68 0.2 0.780">
+        <body name="base" pos="0.72 0.1 0.780">
             <freejoint name="base_joint"/>
             <xacro:threepieceassembly_voxel name="base_0_0_0" pos="-0.076 -0.076 0.0" size="0.019 0.019 0.019" density="10000" material="matte_wood_light"/>
@@ -52,5 +52,5 @@
             <xacro:threepieceassembly_voxel name="base_0_4_4" pos="0.076 0.076 0.0" size="0.019 0.019 0.019" density="10000" material="matte_wood_light"/>
         </body>
-        <body name="piece_1" pos="0.68 0.2 0.912" euler="0 0 1.5708">
+        <body name="piece_1" pos="0.72 0.1 0.912" euler="0 0 1.5708">
             <freejoint name="piece_1_joint"/>
             <xacro:threepieceassembly_voxel name="piece_1_0_0_0" pos="-0.034 -0.034 -0.034" size="0.017 0.017 0.017" density="100" material="obj_blue"/>
@@ -70,5 +70,5 @@
             <xacro:threepieceassembly_voxel name="piece_1_2_1_2" pos="0.0 0.034 0.034" size="0.017 0.017 0.017" density="100" material="obj_blue"/>
         </body>
-        <body name="obj" pos="0.68 -0.25 0.841" euler="0 0 1.5708"> <!-- z-axis : 0 0 1.5708 | y-axis : NONE | x-axis : 0 0 1.5708-->
+        <body name="obj" pos="0.72 -0.3 0.841" euler="0 0 1.5708"> <!-- z-axis : 0 0 1.5708 | y-axis : NONE | x-axis : 0 0 1.5708-->
             <freejoint name="obj_joint"/>
             <xacro:threepieceassembly_voxel name="piece_2_0_0_0" pos="-0.04 -0.04 -0.06" size="0.02 0.02 0.02" density="100" material="obj_red"/>

File: fr3_husky_description/mjcf/yaw_scene.xml.xacro (robot description, xacro)
@@ -7,5 +7,5 @@
               group="1" name="wall_rear_visual" material="walls_mat"/> -->
         <!-- Table geometry from robosuite TableArena with NutAssembly dimensions -->
-        <body name="table" pos="0.7 -0.25 0.6">
+        <body name="table" pos="0.9 -0.05 0.6">
             <geom name="table_collision"
                   pos="0 0 0"
@@ -57,6 +57,6 @@
         </body>
 <!-- Movable T-shaped object -->
-<body name="obj" pos="0.70 -0.50 0.84" quat="1 0 0 0">
-    <joint name="obj_joint" type="free" damping="0.0005"/>
+<body name="obj" pos="0.78 -0.35 0.84" quat="1 0 0 0">
+      <freejoint name="obj_joint"/>
     <geom name="obj_t_stem"
           type="box"
@@ -79,5 +79,5 @@
 </body>
 <!-- Fixed T-shaped socket with small clearance -->
-<body name="t_slot_fixture" pos="0.70 -0.25 0.65" quat="1 0 0 0">
+<body name="t_slot_fixture" pos="0.78 -0.10 0.65" quat="1 0 0 0">
     <geom name="t_slot_floor"
           type="box"

Commit message: re-arrange the object position in each scene

File: fr3_husky_description/mjcf/coffee_scene.xml.xacro (robot description, xacro)
@@ -204,5 +204,5 @@
         </body>
         <!-- Coffee pod, which is the manipulated object -->
-        <body name="obj" pos="0.68 -0.3 0.7" quat="1 0 0 0"> <!-- z-axis : 1 0 0 0 | y-axis : NONE | x-axis : 1 0 0 0 -->
+        <body name="obj" pos="0.78 -0.28 0.65" quat="1 0 0 0"> <!-- z-axis : 1 0 0 0 | y-axis : NONE | x-axis : 1 0 0 0 -->
             <freejoint name="obj_joint"/>
             <geom name="coffee_pod_g0"

File: fr3_husky_description/mjcf/dual_fr3_husky_yaw.xml.xacro (robot description, xacro)
@@ -190,11 +190,5 @@
         <!-- ground plane -->
         <geom name="floor" type="plane" size="0 0 0.05" material="floorplane" />
-        <!-- <camera name="front_overview"
-                mode="fixed"
-                pos="1.15 -0.25 1.15"
-                euler="0 0.9 1.57"
-                fovy="55"
-                resolution="640 480" /> -->
-        <xacro:square_scene/>
+        <xacro:yaw_scene/>
         <body name="root" pos="0 0 0">
             <joint name="world_joint" type="free" stiffness="0" damping="0" frictionloss="0" armature="0" />

File: fr3_husky_description/mjcf/square_scene.xml.xacro (robot description, xacro)
@@ -72,5 +72,5 @@
         </body>
         <!-- Square nut from robosuite square-nut.xml --> <!-- z-axis : 0.7071 0 0 -0.7071 | y-axis : 0.7071 0 0 -0.7071 | x-axis : 0.7071 0 0 -0.7071 -->
-        <body name="obj" pos="0.72 -0.3 0.62" quat="0.7071 0 0 -0.7071">
+        <body name="obj" pos="0.78 -0.28 0.65" quat="0.7071 0 0 -0.7071">
             <freejoint name="obj_joint"/>
             <geom pos="-0.03325 0 0"

File: fr3_husky_description/mjcf/threading_scene.xml.xacro (robot description, xacro)
@@ -17,9 +17,9 @@
             <geom name="threading_table_top"
                   type="box"
-                  size="0.26 0.5 0.02"
+                  size="0.26 0.55 0.02"
                   material="table_ceramic"
                   friction="1 0.005 0.0001"/>
         </body>
-        <body name="obj" pos="0.68 -0.4 0.8" quat="0 0 0 1"> <!-- z-axis : 0 0 0 1 | y-axis : NONE | x-axis : 0 0 0 1-->
+        <body name="obj" pos="0.78 -0.32 0.75" quat="0 0 0 1"> <!-- z-axis : 0 0 0 1 | y-axis : NONE | x-axis : 0 0 0 1-->
             <freejoint name="obj_joint"/>
             <geom name="obj_needle"
@@ -41,5 +41,5 @@
                   solimp="0.9 0.95 0.001"/>
         </body>
-        <body name="tripod_obj" pos="0.80 -0.05 0.8" quat="0.7071068 0 0 0.7071068">
+        <body name="tripod_obj" pos="0.80 0.05 0.8" quat="0.7071068 0 0 0.7071068">
             <geom name="tripod_obj_ring_0" type="box" pos="0 -0.015 0.073" size="0.02 0.0062 0.0062" material="obj_blue" density="100" friction="0.3 0.005 0.0001" solref="0.02 1" solimp="0.9 0.95 0.001"/>
             <geom name="tripod_obj_ring_1" type="box" pos="0 -0.009 0.073" size="0.02 0.0062 0.0062" material="obj_blue" density="100" friction="0.3 0.005 0.0001" solref="0.02 1" solimp="0.9 0.95 0.001"/>

File: fr3_husky_description/mjcf/threepieceassembly_scene.xml.xacro (robot description, xacro)
@@ -33,5 +33,5 @@
                   solimp="0.9 0.95 0.001"/>
         </body>
-        <body name="base" pos="0.72 0.1 0.780">
+        <body name="base" pos="0.72 0.1 0.67">
             <freejoint name="base_joint"/>
             <xacro:threepieceassembly_voxel name="base_0_0_0" pos="-0.076 -0.076 0.0" size="0.019 0.019 0.019" density="10000" material="matte_wood_light"/>
@@ -52,5 +52,5 @@
             <xacro:threepieceassembly_voxel name="base_0_4_4" pos="0.076 0.076 0.0" size="0.019 0.019 0.019" density="10000" material="matte_wood_light"/>
         </body>
-        <body name="piece_1" pos="0.72 0.1 0.912" euler="0 0 1.5708">
+        <body name="piece_1" pos="0.72 0.1 0.70" euler="0 0 1.5708">
             <freejoint name="piece_1_joint"/>
             <xacro:threepieceassembly_voxel name="piece_1_0_0_0" pos="-0.034 -0.034 -0.034" size="0.017 0.017 0.017" density="100" material="obj_blue"/>
@@ -70,5 +70,5 @@
             <xacro:threepieceassembly_voxel name="piece_1_2_1_2" pos="0.0 0.034 0.034" size="0.017 0.017 0.017" density="100" material="obj_blue"/>
         </body>
-        <body name="obj" pos="0.72 -0.3 0.841" euler="0 0 1.5708"> <!-- z-axis : 0 0 1.5708 | y-axis : NONE | x-axis : 0 0 1.5708-->
+        <body name="obj" pos="0.78 -0.28 0.75" euler="0 0 1.5708"> <!-- z-axis : 0 0 1.5708 | y-axis : NONE | x-axis : 0 0 1.5708-->
             <freejoint name="obj_joint"/>
             <xacro:threepieceassembly_voxel name="piece_2_0_0_0" pos="-0.04 -0.04 -0.06" size="0.02 0.02 0.02" density="100" material="obj_red"/>

File: fr3_husky_description/mjcf/yaw_scene.xml.xacro (robot description, xacro)
@@ -1,5 +1,5 @@
 <?xml version="1.0" encoding="utf-8"?>
 <mujoco xmlns:xacro="http://www.ros.org/wiki/xacro">
-    <xacro:macro name="square_scene">
+    <xacro:macro name="yaw_scene">
         <!-- Visual walls from robosuite PegsArena -->
         <!-- <geom pos="-1.2 0 1.5" quat="0.5 0.5 0.5 0.5"
@@ -10,5 +10,5 @@
             <geom name="table_collision"
                   pos="0 0 0"
-                  size="0.4 0.6 0.025"
+                  size="0.4 0.65 0.025"
                   type="box"
                   group="0"
@@ -16,5 +16,5 @@
             <geom name="table_visual"
                   pos="0 0 0"
-                  size="0.4 0.6 0.025"
+                  size="0.4 0.65 0.025"
                   type="box"
                   conaffinity="0"
@@ -57,5 +57,5 @@
         </body>
 <!-- Movable T-shaped object -->
-<body name="obj" pos="0.78 -0.35 0.84" quat="1 0 0 0">
+<body name="obj" pos="0.78 -0.4 0.65" quat="1 0 0 0">
       <freejoint name="obj_joint"/>
     <geom name="obj_t_stem"
@@ -79,5 +79,5 @@
 </body>
 <!-- Fixed T-shaped socket with small clearance -->
-<body name="t_slot_fixture" pos="0.78 -0.10 0.65" quat="1 0 0 0">
+<body name="t_slot_fixture" pos="0.78 0.05 0.65" quat="1 0 0 0">
     <geom name="t_slot_floor"
           type="box"

Commit message: minor color change

File: fr3_husky_description/mjcf/coffee_scene.xml.xacro (robot description, xacro)
@@ -70,5 +70,5 @@
                       condim="4"
                       rgba="0.13 0.13 0.13 1"
-                      material="ceramic"/>
+                      material="matte_black"/>
             </body>
             <body name="coffee_machine_lid_main" pos="0 0.0385 0.144105" quat="0.5 0.8660254 0 0">
@@ -84,5 +84,5 @@
                       condim="4"
                       rgba="0.839 0.839 0.839 1"
-                      material="ceramic"/>
+                      material="matte_ivory"/>
             </body>
             <body name="coffee_machine_base_root" pos="0 0.0 -0.1055" quat="0 0 0 1">
@@ -98,5 +98,5 @@
                       condim="4"
                       rgba="0.13 0.13 0.13 1"
-                      material="ceramic"/>
+                      material="matte_black"/>
             </body>
             <body name="coffee_machine_pod_holder_holder_root" pos="0 0.06355 0.0865">

File: fr3_husky_description/mjcf/dual_fr3_husky_coffee.xml.xacro (robot description, xacro)
@@ -174,8 +174,11 @@
         <texture file="$(find fr3_husky_description)/textures/white-space.png" type="2d" name="tex-white-space"/>
         <texture file="$(find fr3_husky_description)/textures/white-wood.png" type="2d" name="tex-white-wood"/>
+        <texture file="$(find fr3_husky_description)/textures/bleached-wood.png" type="2d" name="tex-bleached-wood"/>
         <material name="obj_red" rgba="0.72 0.28 0.25 1" specular="0.02" shininess="0.02" reflectance="0.0" texture="tex-white-space"/>
         <material name="obj_blue" rgba="0.28 0.42 0.72 1" specular="0.02" shininess="0.02" reflectance="0.0" texture="tex-white-space"/>
         <material name="obj_green" rgba="0.32 0.60 0.38 1" specular="0.02" shininess="0.02" reflectance="0.0" texture="tex-white-space"/>
         <material name="obj_yellow" rgba="0.78 0.66 0.25 1" specular="0.02" shininess="0.02" reflectance="0.0" texture="tex-white-space"/>
+        <material name="matte_black" rgba="0.13 0.13 0.13 1" specular="0.02" shininess="0.02" reflectance="0.0" texture="tex-bleached-wood"/>
+        <material name="matte_ivory" rgba="0.839 0.839 0.839 1" specular="0.02" shininess="0.02" reflectance="0.0" texture="tex-bleached-wood"/>
         <material name="matte_wood_dark" rgba="0.47 0.39 0.30 1" specular="0.02" shininess="0.02" reflectance="0.0" texture="tex-white-wood"/>
         <material name="matte_wood_light" rgba="0.72 0.62 0.51 1" specular="0.02" shininess="0.02" reflectance="0.0" texture="tex-white-wood"/>
