Commit message: changes

File: fr3_husky_description/robots/dual_fr3.srdf.xacro (robot description, xacro)
@@ -15,5 +15,6 @@
                            ee_id="franka_hand"
                            no_prefix="false"
-                           arm_prefix="left_">
+                           arm_prefix="left_"
+                           include_virtual_joint="false">
     </xacro:franka_arm_srdf>
     <xacro:franka_arm_srdf arm_id="fr3"
@@ -21,5 +22,6 @@
                            ee_id="franka_hand"
                            no_prefix="false"
-                           arm_prefix="right_">
+                           arm_prefix="right_"
+                           include_virtual_joint="false">
     </xacro:franka_arm_srdf>
     <xacro:if value="$(arg with_sc)"> <!-- if sc -->

File: fr3_husky_description/robots/dual_fr3_husky.srdf.xacro (robot description, xacro)
@@ -18,5 +18,6 @@
                            ee_id="franka_hand"
                            no_prefix="false"
-                           arm_prefix="left_">
+                           arm_prefix="left_"
+                           include_virtual_joint="false">
     </xacro:franka_arm_srdf>
     <xacro:franka_arm_srdf arm_id="fr3"
@@ -24,5 +25,6 @@
                            ee_id="franka_hand"
                            no_prefix="false"
-                           arm_prefix="right_">
+                           arm_prefix="right_"
+                           include_virtual_joint="false">
     </xacro:franka_arm_srdf>
     <xacro:if value="$(arg with_sc)"> <!-- if sc -->
@@ -719,5 +721,5 @@
     <disable_collisions link1="right_fr3_link5" link2="rear_left_wheel${wheel_suffix}"   reason="Never"/>
     <!-- base - base -->
-    <xacro:husky_base_srdf/>
+    <xacro:husky_base_srdf base_link="base_link"/>
     <!-- left link - right link -->
     <disable_collisions link1="left_fr3_link0" link2="right_fr3_link0" reason="Adjacent"/>

File: fr3_husky_description/robots/husky_base.srdf.xacro (robot description, xacro)
@@ -1,17 +1,17 @@
 <?xml version='1.0' encoding='utf-8'?>
 <robot xmlns:xacro="http://www.ros.org/wiki/xacro" >
-    <xacro:macro name="husky_base_srdf">
+    <xacro:macro name="husky_base_srdf" params="base_link:='mobile_base'">
         <disable_collisions link1="front_left_wheel"  link2="front_right_wheel"  reason="Never"/>
-        <disable_collisions link1="front_left_wheel"  link2="mobile_base"        reason="Adjacent"/>
+        <disable_collisions link1="front_left_wheel"  link2="${base_link}"       reason="Adjacent"/>
         <disable_collisions link1="front_left_wheel"  link2="rear_left_wheel"    reason="Never"/>
         <disable_collisions link1="front_left_wheel"  link2="rear_right_wheel"   reason="Never"/>
         <disable_collisions link1="front_left_wheel"  link2="top_structure_link" reason="Never"/>
-        <disable_collisions link1="front_right_wheel" link2="mobile_base"        reason="Adjacent"/>
+        <disable_collisions link1="front_right_wheel" link2="${base_link}"       reason="Adjacent"/>
         <disable_collisions link1="front_right_wheel" link2="rear_left_wheel"    reason="Never"/>
         <disable_collisions link1="front_right_wheel" link2="rear_right_wheel"   reason="Never"/>
         <disable_collisions link1="front_right_wheel" link2="top_structure_link" reason="Never"/>
-        <disable_collisions link1="mobile_base"       link2="rear_left_wheel"    reason="Adjacent"/>
-        <disable_collisions link1="mobile_base"       link2="rear_right_wheel"   reason="Adjacent"/>
-        <disable_collisions link1="mobile_base"       link2="top_structure_link" reason="Adjacent"/>
+        <disable_collisions link1="${base_link}"      link2="rear_left_wheel"    reason="Adjacent"/>
+        <disable_collisions link1="${base_link}"      link2="rear_right_wheel"   reason="Adjacent"/>
+        <disable_collisions link1="${base_link}"      link2="top_structure_link" reason="Adjacent"/>
         <disable_collisions link1="rear_left_wheel"   link2="rear_right_wheel"   reason="Never"/>
         <disable_collisions link1="rear_right_wheel"  link2="top_structure_link" reason="Never"/>

File: fr3_husky_description/robots/single_fr3.srdf.xacro (robot description, xacro)
@@ -20,5 +20,6 @@
                            ee_id="franka_hand"
                            no_prefix="false"
-                           arm_prefix="${modified_prefix}">
+                           arm_prefix="${modified_prefix}"
+                           include_virtual_joint="false">
     </xacro:franka_arm_srdf>
     <xacro:if value="$(arg with_sc)">

File: fr3_husky_description/robots/single_fr3_husky.srdf.xacro (robot description, xacro)
@@ -23,5 +23,6 @@
                            ee_id="franka_hand"
                            no_prefix="false"
-                           arm_prefix="${modified_prefix}">
+                           arm_prefix="${modified_prefix}"
+                           include_virtual_joint="false">
     </xacro:franka_arm_srdf>
     <xacro:if value="$(arg with_sc)">

Commit message: save.

File: fr3_husky_description/robots/dual_fr3.srdf.xacro (robot description, xacro)
@@ -15,6 +15,5 @@
                            ee_id="franka_hand"
                            no_prefix="false"
-                           arm_prefix="left_"
-                           include_virtual_joint="false">
+                           arm_prefix="left_">
     </xacro:franka_arm_srdf>
     <xacro:franka_arm_srdf arm_id="fr3"
@@ -22,6 +21,5 @@
                            ee_id="franka_hand"
                            no_prefix="false"
-                           arm_prefix="right_"
-                           include_virtual_joint="false">
+                           arm_prefix="right_">
     </xacro:franka_arm_srdf>
     <xacro:if value="$(arg with_sc)"> <!-- if sc -->
